File: assets/kim-demo/KIM Demo.kicad_sch (KiCad schematic)
At the start: 24 parts, among them J1 6502 BUS, U1 74HC04, U2 74HC00, U3 74HC138, U4 74HC373

Commit message: KIM Demo: draw it for the KIM Board's breadboard headers
The sheet (now Rev 1.1) takes the bus from the KIM Board's breadboard
headers instead of a 2x20 header: J1 is Row 1 (the 6502 BUS's odd pins)
and J2 is Row 2 (its even pins), every pin labelled, with a note mapping
the rows back to the bus.

Two fixes carried over from the retired LED Accessory copy (6502-KIM
32b9900):

- The header's supply was labelled 5V, a separate net from the chips'
  VCC, so on paper nothing powered the chips. It is VCC now.
- The LEDs are renumbered so the latch's output n drives R(n+1) and
  D(n+1), in the order the series shows them.

The netlist is otherwise unchanged: the latch still loads only on a
write to $9400-$97FF. ERC has the same 77 label-style warnings as
before. The empty PCB file goes: this circuit is built on a breadboard
and has no PCB. The KIM page now says "jumper wires from the bus",
which is true of today's KIM and the KIM Board alike.

Co-Authored-By: Claude Opus 5.5 <noreply@anthropic.com>
Parts:
- removed J1: 6502 BUS, symbol Connector_Generic:Conn_02x20_Odd_Even
- added J1: ROW 1, symbol Connector_Generic:Conn_01x20
- added J2: ROW 2, symbol Connector_Generic:Conn_01x20
- renumbered D5 to D2, D2 to D3, D6 to D4, D3 to D5, D7 to D6, D4 to D7
Connections:
- net A0: now also J2.19 (Pin_19)
- net A1: now also J2.18 (Pin_18)
- net A10: now also J2.9 (Pin_9)
- net A11: now also J2.8 (Pin_8)
- net A12: now also J2.7 (Pin_7)
- net A13: now also J2.6 (Pin_6)
- net A14: now also J2.5 (Pin_5)
- net A15: now also J2.4 (Pin_4)
- net A2: now also J2.17 (Pin_17)
- net A3: now also J2.16 (Pin_16)
- net A4: now also J2.15 (Pin_15)
- net A5: now also J2.14 (Pin_14)
- net A6: now also J2.13 (Pin_13)
- net A7: now also J2.12 (Pin_12)
- net A8: now also J2.11 (Pin_11)
- net A9: now also J2.10 (Pin_10)
- net BE: now also J1.6 (Pin_6)
- net D0: now also J1.19 (Pin_19)
- net D1: now also J1.18 (Pin_18)
- net D2: now also J1.17 (Pin_17)
- net D3: now also J1.16 (Pin_16)
- net D4: now also J1.15 (Pin_15)
- net D5: now also J1.14 (Pin_14)
- net D6: now also J1.13 (Pin_13)
- net D7: now also J1.12 (Pin_12)
- net EXP0: now also J2.3 (Pin_3)
- net EXP1: now also J2.2 (Pin_2)
- net EXP2: now also J1.11 (Pin_11)
- net EXP3: now also J1.10 (Pin_10)
- net GND: now also J1.1 (Pin_1), J2.20 (Pin_20)
- net IRQB: now also J1.3 (Pin_3)
- net NMIB: now also J1.4 (Pin_4)
- net PHI2: now also J1.9 (Pin_9)
- net RDY: now also J1.5 (Pin_5)
- net RESB: now also J1.2 (Pin_2)
- net RWB: now also J1.7 (Pin_7)
- net SYNC: now also J1.8 (Pin_8)
- net VCC: now also J1.20 (Pin_20), J2.1 (Pin_1)
Other:
- note added: "Breadboard headers (KIM Board) Row 1 = 6502 BUS odd pins, Row 2 = even pins"
